File: Teensy macro pad.kicad_sch (KiCad schematic)
At the start: 49 parts, among them J1 USB_C_Receptacle_USB2.0_14P, J2 AVR-ISP-6, J3 Conn_01x05_Pin, SW0,0 CherryMX, SW0,1 CherryMX, SW0,2 CherryMX, SW0,3 CherryMX, SW0,4 CherryMX, SW1 SW_Push, SW1,0 CherryMX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

Commit message: Rename reset switch symbol
Having a switch with reference SW1 as well as ones with SW1,0 to SW1,4
seemed to confuse Fabrication Toolkit or JLCPCB's BOM processor.
Parts:
- renumbered SW1 to SWR1
Changed lines of the file:
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@@
 		(dnp no)
 		(fields_autoplaced yes)
-		(property "Reference" "SW1"
+		(property "Reference" "SWR1"
 			(at 118.11 29.21 0)
 			(effects
@@
 			(project ""
 				(path "/bcf4c563-ed90-4192-81fd-782593c0996d"
-					(reference "SW1")
+					(reference "SWR1")
 					(unit 1)
 				)
